Commit message: pkg working

File: description/urdf/model.gazebo.xacro (robot description, xacro)
@@ -3,4 +3,43 @@
   <xacro:arg name="laser_visual" default="false"/>
   <xacro:arg name="imu_visual"   default="false"/>
+  <gazebo reference="base_link">
+    <material>Gazebo/DarkGrey</material>
+  </gazebo>
+  <gazebo reference="wheel_left_link">
+    <mu1>0.1</mu1>
+    <mu2>0.1</mu2>
+    <kp>500000.0</kp>
+    <kd>10.0</kd>
+    <minDepth>0.001</minDepth>
+    <maxVel>0.1</maxVel>
+    <fdir1>1 0 0</fdir1>
+    <material>Gazebo/FlatBlack</material>
+  </gazebo>
+  <gazebo reference="wheel_right_link">
+    <mu1>0.1</mu1>
+    <mu2>0.1</mu2>
+    <kp>500000.0</kp>
+    <kd>10.0</kd>
+    <minDepth>0.001</minDepth>
+    <maxVel>0.1</maxVel>
+    <fdir1>1 0 0</fdir1>
+    <material>Gazebo/FlatBlack</material>
+  </gazebo>
+  <gazebo reference="caster_back_link">
+    <mu1>0.1</mu1>
+    <mu2>0.1</mu2>
+    <kp>1000000.0</kp>
+    <kd>100.0</kd>
+    <minDepth>0.001</minDepth>
+    <maxVel>1.0</maxVel>
+    <material>Gazebo/FlatBlack</material>
+  </gazebo>
+  <gazebo reference="imu_link">
+    <sensor type="imu" name="imu">
+      <always_on>true</always_on>
+      <visualize>$(arg imu_visual)</visualize>
+    </sensor>
+    <material>Gazebo/FlatBlack</material>
+  </gazebo>
   <gazebo>
     <plugin name="model_controller" filename="libgazebo_ros_diff_drive.so">
@@ -8,9 +47,12 @@
       <odometryTopic>odom</odometryTopic>
       <odometryFrame>odom</odometryFrame>
+      <odometrySource>world</odometrySource>
+      <publishOdomTF>true</publishOdomTF>
       <robotBaseFrame>base_footprint</robotBaseFrame>
       <publishWheelTF>false</publishWheelTF>
+      <publishTf>true</publishTf>
       <publishWheelJointState>true</publishWheelJointState>
       <legacyMode>false</legacyMode>
-      <updateRate>100</updateRate>
+      <updateRate>30</updateRate>
       <leftJoint>wheel_left_joint</leftJoint>
       <rightJoint>wheel_right_joint</rightJoint>
@@ -19,37 +61,6 @@
       <wheelAcceleration>1</wheelAcceleration>
       <wheelTorque>10</wheelTorque>
+      <rosDebugLevel>na</rosDebugLevel>
     </plugin>
-  </gazebo>
-  <gazebo reference="base_link">
-    <material>Gazebo/Grey</material>
-  </gazebo>
-  <gazebo reference="wheel_left_link">
-    <mu1>10</mu1>
-    <mu2>10</mu2>
-    <kp>500000.0</kp>
-    <kd>10.0</kd>
-    <minDepth>0.001</minDepth>
-    <maxVel>0.1</maxVel>
-    <fdir1>1 0 0</fdir1>
-    <material>Gazebo/DarkGrey</material>
-  </gazebo>
-  <gazebo reference="wheel_right_link">
-    <mu1>10</mu1>
-    <mu2>10</mu2>
-    <kp>500000.0</kp>
-    <kd>10.0</kd>
-    <minDepth>0.001</minDepth>
-    <maxVel>0.1</maxVel>
-    <fdir1>1 0 0</fdir1>
-    <material>Gazebo/DarkGrey</material>
-  </gazebo>
-  <gazebo reference="caster_back_link">
-    <mu1>0.0</mu1>
-    <mu2>0.0</mu2>
-    <kp>1000000.0</kp>
-    <kd>100.0</kd>
-    <minDepth>0.001</minDepth>
-    <maxVel>1.0</maxVel>
-    <material>Gazebo/Grey</material>
   </gazebo>
   <gazebo>
@@ -57,8 +68,9 @@
       <alwaysOn>true</alwaysOn>
       <bodyName>imu_link</bodyName>
-      <topicName>/imu</topicName>
-      <serviceName>/imu_service</serviceName>
+      <frameName>imu_link</frameName>
+      <topicName>imu</topicName>
+      <serviceName>imu_service</serviceName>
       <gaussianNoise>0.0</gaussianNoise>
-      <updateRate>100.0</updateRate>
+      <updateRate>200</updateRate>
       <imu>
         <noise>
@@ -80,18 +92,10 @@
     </plugin>
   </gazebo>
-  <gazebo reference="imu_link">
-    <sensor type="imu" name="imu">
-      <always_on>true</always_on>
-      <update_rate>50</update_rate>
-      <visualize>$(arg imu_visual)</visualize>
-    </sensor>
-    <material>Gazebo/Grey</material>
-  </gazebo>
   <gazebo reference="base_scan">
-    <material>Gazebo/DarkGrey</material>
+    <material>Gazebo/FlatBlack</material>
     <sensor type="ray" name="lds_lfcd_sensor">
       <pose>0 0 0 0 0 0</pose>
       <visualize>$(arg laser_visual)</visualize>
-      <update_rate>1800</update_rate>
+      <update_rate>5</update_rate>
       <ray>
         <scan>
@@ -100,5 +104,5 @@
             <resolution>1</resolution>
             <min_angle>0.0</min_angle>
-            <max_angle>6.28</max_angle>
+            <max_angle>6.28319</max_angle>
           </horizontal>
         </scan>
@@ -115,5 +119,5 @@
       </ray>
       <plugin name="gazebo_ros_lds_lfcd_controller" filename="libgazebo_ros_laser.so">
-        <topicName>/scan</topicName>
+        <topicName>scan</topicName>
         <frameName>base_scan</frameName>
       </plugin>

File: description/urdf/model.urdf.xacro (robot description, xacro)
@@ -20,13 +20,13 @@
       <origin xyz="-0.032 0 0.070" rpy="0 0 0"/>
       <geometry>
-        <box size="0.140 0.140 0.140"/>
+        <box size="0.140 0.140 0.143"/>
       </geometry>
     </collision>
     <inertial>
-      <origin xyz="-0.032 0 0" rpy="0 0 0"/>
-      <mass value="1"/>
-      <inertia ixx="0.01" ixy="0.0" ixz="0.0"
-               iyy="0.01" iyz="0.0"
-               izz="0.01" />
+      <origin xyz="0 0 0" rpy="0 0 0"/>
+      <mass value="8.2573504e-01"/>
+      <inertia ixx="2.2124416e-03" ixy="-1.2294101e-05" ixz="3.4938785e-05"
+               iyy="2.1193702e-03" iyz="-5.0120904e-06"
+               izz="2.0064271e-03" />
     </inertial>
   </link>
@@ -34,10 +34,10 @@
     <parent link="base_link"/>
     <child link="wheel_left_link"/>
-    <origin xyz="0.0 0.08 0.023" rpy="${-M_PI*0.5} 0 0"/>
+    <origin xyz="0.0 0.08 0.023" rpy="-1.57 0 0"/>
     <axis xyz="0 0 1"/>
   </joint>
   <link name="wheel_left_link">
     <visual>
-      <origin xyz="0 0 0" rpy="${M_PI*0.5} 0 0"/>
+      <origin xyz="0 0 0" rpy="1.57 0 0"/>
       <geometry>
         <mesh filename="package://description/meshes/wheels/left_tire.stl" scale="0.001 0.001 0.001"/>
@@ -53,19 +53,19 @@
     <inertial>
       <origin xyz="0 0 0" />
-      <mass value="0.01" />
-      <inertia ixx="0.001" ixy="0.0" ixz="0.0"
-               iyy="0.001" iyz="0.0"
-               izz="0.001" />
-    </inertial>
+      <mass value="2.8498940e-02" />
+      <inertia ixx="1.1175580e-05" ixy="-4.2369783e-11" ixz="-5.9381719e-09"
+               iyy="1.1192413e-05" iyz="-1.4400107e-11"
+               izz="2.0712558e-05" />
+      </inertial>
   </link>
   <joint name="wheel_right_joint" type="continuous">
     <parent link="base_link"/>
     <child link="wheel_right_link"/>
-    <origin xyz="0.0 -0.08 0.023" rpy="${-M_PI*0.5} 0 0"/>
+    <origin xyz="0.0 -0.080 0.023" rpy="-1.57 0 0"/>
     <axis xyz="0 0 1"/>
   </joint>
   <link name="wheel_right_link">
     <visual>
-      <origin xyz="0 0 0" rpy="${M_PI*0.5} 0 0"/>
+      <origin xyz="0 0 0" rpy="1.57 0 0"/>
       <geometry>
         <mesh filename="package://description/meshes/wheels/right_tire.stl" scale="0.001 0.001 0.001"/>
@@ -81,25 +81,25 @@
     <inertial>
       <origin xyz="0 0 0" />
-      <mass value="0.01" />
-      <inertia ixx="0.001" ixy="0.0" ixz="0.0"
-               iyy="0.001" iyz="0.0"
-               izz="0.001" />
-    </inertial>
+      <mass value="2.8498940e-02" />
+      <inertia ixx="1.1175580e-05" ixy="-4.2369783e-11" ixz="-5.9381719e-09"
+               iyy="1.1192413e-05" iyz="-1.4400107e-11"
+               izz="2.0712558e-05" />
+      </inertial>
   </link>
   <joint name="caster_back_joint" type="fixed">
     <parent link="base_link"/>
     <child link="caster_back_link"/>
-    <origin xyz="-0.081 0 -0.004" rpy="${-M_PI*0.5} 0 0"/>
+    <origin xyz="-0.081 0 -0.004" rpy="-1.57 0 0"/>
   </joint>
   <link name="caster_back_link">
     <collision>
-      <origin xyz="0 0 0" rpy="0 0 0"/>
+      <origin xyz="0 0.001 0" rpy="0 0 0"/>
       <geometry>
-        <box size="0.030 0.010 0.020"/>
+        <box size="0.030 0.009 0.020"/>
       </geometry>
     </collision>
     <inertial>
       <origin xyz="0 0 0" />
-      <mass value="0.01" />
+      <mass value="0.005" />
       <inertia ixx="0.001" ixy="0.0" ixz="0.0"
                iyy="0.001" iyz="0.0"
@@ -116,5 +116,5 @@
     <parent link="base_link"/>
     <child link="base_scan"/>
-    <origin xyz="-0.032 0 0.171" rpy="0 0 0"/>
+    <origin xyz="-0.032 0 0.172" rpy="0 0 0"/>
   </joint>
   <link name="base_scan">
@@ -127,11 +127,11 @@
     </visual>
     <collision>
-      <origin xyz="0 0 0" rpy="0 0 0"/>
+      <origin xyz="0.015 0 -0.0065" rpy="0 0 0"/>
       <geometry>
-        <cylinder length="0.0408" radius="0.070"/>
+        <cylinder length="0.0315" radius="0.055"/>
       </geometry>
     </collision>
     <inertial>
-      <mass value="0.01" />
+      <mass value="0.114" />
       <origin xyz="0 0 0" />
       <inertia ixx="0.001" ixy="0.0" ixz="0.0"

Commit message: d435 sensor added

File: description/urdf/model.gazebo.xacro (robot description, xacro)
@@ -42,4 +42,5 @@
     <material>Gazebo/FlatBlack</material>
   </gazebo>
+  <!-- Controller -->
   <gazebo>
     <plugin name="model_controller" filename="libgazebo_ros_diff_drive.so">
@@ -64,4 +65,5 @@
     </plugin>
   </gazebo>
+  <!-- IMU sensor -->
   <gazebo>
     <plugin name="imu_plugin" filename="libgazebo_ros_imu.so">
@@ -92,4 +94,5 @@
     </plugin>
   </gazebo>
+  <!-- LiDAR sensor -->
   <gazebo reference="base_scan">
     <material>Gazebo/FlatBlack</material>
@@ -124,3 +127,60 @@
     </sensor>
   </gazebo>
+  <!-- d435 sensor -->
+  <gazebo reference="camera_frame">
+      <sensor type="depth" name="d435_depth_frame_sensor">
+      <update_rate>20.0</update_rate>
+      <camera name="d435_depth_camera">
+          <horizontal_fov>1.3962634</horizontal_fov>
+          <image>
+          <width>1280</width>
+          <height>720</height>
+          <format>R8G8B8</format>
+          </image>
+          <clip>
+          <near>0.02</near>
+          <far>100</far>
+          </clip>
+          <noise>
+          <type>gaussian</type>
+          <mean>0.0</mean>
+          <stddev>0.007</stddev>
+          </noise>
+      </camera>
+      <plugin name="d435_depth_frame_controller" filename="libgazebo_ros_openni_kinect.so">
+          <alwaysOn>true</alwaysOn>
+          <updateRate>20.0</updateRate>
+          <imageTopicName>camera/rgb/image_raw</imageTopicName>
+          <depthImageTopicName>camera/depth/image_raw</depthImageTopicName>
+          <cameraInfoTopicName>camera/rgb/camera_info</cameraInfoTopicName>
+          <depthImageInfoTopicName>camera/depth/camera_info</depthImageInfoTopicName>
+          <pointCloudTopicName>camera/depth/points</pointCloudTopicName>
+          <frameName>d435_depth_optical_frame</frameName>
+          <hackBaseline>0.07</hackBaseline>
+          <distortion_k1>0.00000001</distortion_k1>
+          <distortion_k2>0.00000001</distortion_k2>
+          <distortion_k3>0.00000001</distortion_k3>
+          <distortion_t1>0.00000001</distortion_t1>
+          <distortion_t2>0.00000001</distortion_t2>
+      </plugin>
+      </sensor>
+  </gazebo>
+  <!-- Planar -->
+  <gazebo>
+      <plugin name="dummy_drive" filename="libgazebo_ros_planar_move.so">
+          <legacyMode>false</legacyMode>
+          <alwaysOn>true</alwaysOn>
+          <updateRate>100</updateRate>
+          <covariance_x>0.000100</covariance_x>
+          <covariance_y>0.000100</covariance_y>
+          <covariance_yaw>0.010000</covariance_yaw>
+          <broadcastTF>100</broadcastTF>
+          <torque>5</torque>
+          <commandTopic>cmd_vel</commandTopic>
+          <odometryTopic>odom</odometryTopic>
+          <odometryFrame>odom</odometryFrame>
+          <odometryRate>100.0</odometryRate>
+          <robotBaseFrame>base_footprint</robotBaseFrame>
+      </plugin>
+  </gazebo>
 </robot>

File: description/urdf/model.urdf.xacro (robot description, xacro)
@@ -3,5 +3,7 @@
   <xacro:include filename="$(find description)/urdf/common_properties.xacro"/>
   <xacro:include filename="$(find description)/urdf/model.gazebo.xacro"/>
+  <!-- Base footprint -->
   <link name="base_footprint"/>
+  <!-- Base link -->
   <joint name="base_joint" type="fixed">
     <parent link="base_footprint"/>
@@ -31,4 +33,5 @@
     </inertial>
   </link>
+  <!-- Wheel left -->
   <joint name="wheel_left_joint" type="continuous">
     <parent link="base_link"/>
@@ -59,4 +62,5 @@
       </inertial>
   </link>
+  <!-- Wheel right -->
   <joint name="wheel_right_joint" type="continuous">
     <parent link="base_link"/>
@@ -87,4 +91,5 @@
       </inertial>
   </link>
+  <!-- Caster back -->
   <joint name="caster_back_joint" type="fixed">
     <parent link="base_link"/>
@@ -107,4 +112,5 @@
     </inertial>
   </link>
+  <!-- IMU sensor -->
   <joint name="imu_joint" type="fixed">
     <parent link="base_link"/>
@@ -113,4 +119,5 @@
   </joint>
   <link name="imu_link"/>
+  <!-- LiDAR sensor -->
   <joint name="scan_joint" type="fixed">
     <parent link="base_link"/>
@@ -140,3 +147,34 @@
     </inertial>
   </link>
+  <!-- d435 sensor -->
+  <joint name="camera_joint" type="fixed">
+    <parent link="base_link"/>
+    <child link="camera_link" />
+  </joint>
+  <link name="camera_link">
+    <visual>
+    <origin xyz="0.040 0 0.115" rpy="${M_PI/2} 0 ${M_PI/2}"/>
+      <geometry>
+        <mesh filename="package://description/meshes/sensors/d435.dae" />
+      </geometry>
+      <material name="black"/>
+    </visual>
+    <collision>
+      <origin xyz="0.0 0.0 0.0125" rpy="0 0 0"/>
+      <geometry>
+      <box size="0.02505 0.09 0.025"/>
+      </geometry>
+    </collision>
+    <inertial>
+      <mass value="0.564" />
+      <origin xyz="0 0 0" />
+      <inertia ixx="0.003881243" ixy="0.0" ixz="0.0" iyy="0.000498940" iyz="0.0" izz="0.003879257" />
+    </inertial>
+  </link>
+  <joint name="camera_depth_joint" type="fixed">
+    <parent link="camera_link"/>
+    <child link="camera_frame"/>
+    <origin xyz="0.03 0.0175 0.0125" rpy="0 0 0"/>
+  </joint>
+  <link name="camera_frame"/>
 </robot>
